File: max3421eboard.sch (KiCad schematic (older format))
At the start: 30 parts, among them J1 USB A, J2 USB MicroB, J3 1x10, J4 1x8, J5 1x8, J6 1x3, J7 Conn_01x04, U1 MAX3421E, U2 LP2985-3.3, U3 STMPS2141STR, Y1 12MHz

Commit message: Rescue symbols from cache
Parts:
- U3: symbol Matti:STMPS2151STR -> max3421eboard-rescue:STMPS2151STR-Matti
Changed lines of the file:
@@
 	1750 1550 1750 1400
 $Comp
-L Matti:STMPS2151STR U3
+L max3421eboard-rescue:STMPS2151STR-Matti U3
 U 1 1 5ED2A525
 P 2400 1850
@@
 	2950 1750 3700 1750
 $Comp
-L Matti:VL #PWR0117
+L max3421eboard-rescue:VL-Matti #PWR0117
 U 1 1 5F0C91BD
 P 7850 1250
@@
 $EndComp
 $Comp
-L Matti:VL #PWR0118
+L max3421eboard-rescue:VL-Matti #PWR0118
 U 1 1 5F0CD619
 P 9000 1250
@@
 $EndComp
 $Comp
-L Matti:VL #PWR0125
+L max3421eboard-rescue:VL-Matti #PWR0125
 U 1 1 5F0CF343
 P 6000 1350
@@
 Connection ~ 6000 1350
 $Comp
-L Matti:VL #PWR0126
+L max3421eboard-rescue:VL-Matti #PWR0126
 U 1 1 5F0D8675
 P 6400 3900
@@
 X-
 $Comp
-L Matti:VL #PWR0114
+L max3421eboard-rescue:VL-Matti #PWR0114
 U 1 1 5F28C84A
 P 8200 3650

Commit message: Replace crystal and microUSB connector with the available ones
Parts:
- J2: footprint Connectors:USB_Micro-B_10103594-0001LF -> Connector_USB:USB_Micro-B_Molex-105017-0001
- Y1: footprint Crystals:Crystal_SMD_5032-2pin_5.0x3.2mm_HandSoldering -> Crystal:Crystal_HC49-4H_Vertical
Changed lines of the file:
@@
 F 0 "Y1" H 4800 2382 50  0000 C CNN
 F 1 "12MHz" H 4800 2473 50  0000 C CNN
-F 2 "Crystals:Crystal_SMD_5032-2pin_5.0x3.2mm_HandSoldering" H 4800 2650 50  0001 C CNN
+F 2 "Crystal:Crystal_HC49-4H_Vertical" H 4800 2650 50  0001 C CNN
 F 3 "~" H 4800 2650 50  0001 C CNN
 	1    4800 2650
@@
 F 0 "J2" H 3357 2917 50  0000 C CNN
 F 1 "USB MicroB" H 3357 2826 50  0000 C CNN
-F 2 "Connectors:USB_Micro-B_10103594-0001LF" H 3450 2400 50  0001 C CNN
+F 2 "Connector_USB:USB_Micro-B_Molex-105017-0001" H 3450 2400 50  0001 C CNN
 F 3 "~" H 3450 2400 50  0001 C CNN
 	1    3300 2450
